File: USB-C-power-adapter.kicad_sch (KiCad schematic)
At the start: 0 parts

Commit message: [#57225] Add antmicro logos
Parts:
- added N1: antmicro_logo, antmicro-footprints:antmicro-logo_scaled_12mm_silk, symbol antmicroMechanicalParts:antmicro_logo
- added N2: oshw_logo, antmicro-footprints:OSHW-Logo_5.7x6mm_SilkScreen, symbol antmicroMechanicalParts:oshw_logo
Changed lines of the file:
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@@
+    )
+  )
+  (symbol (lib_id "antmicroMechanicalParts:oshw_logo") (at 119.38 273.05 0) (unit 1)
+    (in_bom no) (on_board yes) (dnp no) (fields_autoplaced)
+    (property "Reference" "N2" (at 125.73 271.0662 0)
+      (effects (font (size 1.27 1.27) (thickness 0.15)) (justify left))
+    )
+    (property "Value" "oshw_logo" (at 125.73 273.6062 0)
+      (effects (font (size 1.27 1.27) (thickness 0.15)) (justify left))
+    )
+    (property "Footprint" "antmicro-footprints:OSHW-Logo_5.7x6mm_SilkScreen" (at 134.62 283.21 0)
+      (effects (font (size 1.27 1.27) (thickness 0.15)) (justify left bottom) hide)
+    )
+    (property "Datasheet" "" (at 134.62 285.75 0)
+      (effects (font (size 1.27 1.27) (thickness 0.15)) (justify left bottom) hide)
+    )
+    (property "Author" "Antmicro" (at 134.62 288.29 0)
+      (effects (font (size 1.27 1.27) (thickness 0.15)) (justify left bottom) hide)
+    )
+    (property "License" "Apache-2.0" (at 134.62 290.83 0)
+      (effects (font (size 1.27 1.27) (thickness 0.15)) (justify left bottom) hide)
+    )
+    (property "MPN" "" (at 119.38 273.05 0)
+      (effects (font (size 1.27 1.27)) hide)
+    )
+    (property "Manufacturer" "" (at 134.62 293.37 0)
+      (effects (font (size 1.27 1.27) (thickness 0.15)) (justify left bottom) hide)
+    )
+    (property "DNP" "" (at 119.38 273.05 0)
+      (effects (font (size 1.27 1.27)))
+    )
+    (instances
+      (project "USB-C-power-adapter"
+        (path "/8da33aa8-79ed-467a-95ed-bf58aa0d1db6"
+          (reference "N2") (unit 1)
+        )
+      )
+    )
+  )
+  (symbol (lib_id "antmicroMechanicalParts:antmicro_logo") (at 96.52 273.05 0) (unit 1)
+    (in_bom no) (on_board yes) (dnp no) (fields_autoplaced)
+    (property "Reference" "N1" (at 102.87 271.0662 0)
+      (effects (font (size 1.27 1.27) (thickness 0.15)) (justify left))
+    )
+    (property "Value" "antmicro_logo" (at 102.87 273.6062 0)
+      (effects (font (size 1.27 1.27) (thickness 0.15)) (justify left))
+    )
+    (property "Footprint" "antmicro-footprints:antmicro-logo_scaled_12mm_silk" (at 111.76 283.21 0)
+      (effects (font (size 1.27 1.27) (thickness 0.15)) (justify left bottom) hide)
+    )
+    (property "Datasheet" "" (at 111.76 285.75 0)
+      (effects (font (size 1.27 1.27) (thickness 0.15)) (justify left bottom) hide)
+    )
+    (property "MPN" "" (at 96.52 273.05 0)
+      (effects (font (size 1.27 1.27)) hide)
+    )
+    (property "Manufacturer" "" (at 111.76 293.37 0)
+      (effects (font (size 1.27 1.27) (thickness 0.15)) (justify left bottom) hide)
+    )
+    (property "Author" "Antmicro" (at 111.76 288.29 0)
+      (effects (font (size 1.27 1.27) (thickness 0.15)) (justify left bottom) hide)
+    )
+    (property "License" "Apache-2.0" (at 111.76 290.83 0)
+      (effects (font (size 1.27 1.27) (thickness 0.15)) (justify left bottom) hide)
+    )
+    (property "DNP" "" (at 96.52 273.05 0)
+      (effects (font (size 1.27 1.27)))
+    )
+    (instances
+      (project "USB-C-power-adapter"
+        (path "/8da33aa8-79ed-467a-95ed-bf58aa0d1db6"
+          (reference "N1") (unit 1)
+        )
+      )
     )
   )

Commit message: [#61462] Update symbols from library and resolve ERC issues
Parts:
- N1: footprint antmicro-footprints:antmicro-logo_scaled_12mm_silk -> antmicro-footprints:antmicro-logo; Public (none) -> False
- N2: footprint antmicro-footprints:OSHW-Logo_5.7x6mm_SilkScreen -> antmicro-footprints:oshw-logo; Public (none) -> False
Changed lines of the file:
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@@
       (effects (font (size 1.27 1.27) (thickness 0.15)) (justify left))
     )
-    (property "Footprint" "antmicro-footprints:OSHW-Logo_5.7x6mm_SilkScreen" (at 134.62 283.21 0)
+    (property "Footprint" "antmicro-footprints:oshw-logo" (at 134.62 283.21 0)
       (effects (font (size 1.27 1.27) (thickness 0.15)) (justify left bottom) hide)
     )
@@
       (effects (font (size 1.27 1.27)))
     )
+    (property "Public" "False" (at 134.62 293.37 0)
+      (effects (font (size 1.27 1.27)) (justify left bottom) hide)
+    )
     (instances
       (project "USB-C-power-adapter"
@@
       (effects (font (size 1.27 1.27) (thickness 0.15)) (justify left))
     )
-    (property "Footprint" "antmicro-footprints:antmicro-logo_scaled_12mm_silk" (at 111.76 283.21 0)
+    (property "Footprint" "antmicro-footprints:antmicro-logo" (at 111.76 283.21 0)
       (effects (font (size 1.27 1.27) (thickness 0.15)) (justify left bottom) hide)
     )
@@
       (effects (font (size 1.27 1.27)))
     )
+    (property "Public" "False" (at 111.76 293.37 0)
+      (effects (font (size 1.27 1.27)) (justify left bottom) hide)
+    )
     (instances
