File: USB-C-power-adapter.kicad_pcb (KiCad board)
At the start: 4 copper layers, 21.9 x 52.5 mm, 124 parts, among them J1 USB-C_GCT_USB4105-GF-A, J2 JST_SH_1x4_SM04B-SRSS-TB-LF-SN, J3 JST_SH_1x4_SM04B-SRSS-TB-LF-SN, J4 Molex_Nano-Fit_1x2_105313-220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, Q1 SQS401EN-T1_BE3, U1 STUSB4500_QFN, U2 SIC477ED-T1-GE3, U3 AP62301Z6-7, U4 AP62301Z6-7, U5 TVS2200DRVR, U6 TPD4E02B04DQA, U7 TVS2200DRVR, U8 TVS2200DRVR

Commit message: [#72550] Update and clenup DRCs
Routing:
- net unconnected-(U6-Pad1): track 0.77 -> 0.00 mm
Other:
- board text added: "USB-C-PD-Adapter Rev ${REVISION} 02/2025 SHA: ########"
- board text removed: "USB-C-PD-Adapter Rev. 1.1.0 07/2024 SHA: ########"
