File: usb-c-power-adapter.kicad_sch (KiCad schematic)
At the start: 0 parts

Commit message: [#72550] Rename project to lower case letters
Other:
- title: USB-C-power-adapter -> usb-c-power-adapter
Changed lines of the file:
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@@
 	(paper "A3")
 	(title_block
-		(title "USB-C-power-adapter")
+		(title "usb-c-power-adapter")
 		(date "2025-02-05")
 		(rev "1.1.1")
@@
 		)
 		(instances
-			(project "USB-C-power-adapter"
+			(project "usb-c-power-adapter"
 				(path "/8da33aa8-79ed-467a-95ed-bf58aa0d1db6"
 					(page "3")
@@
 		)
 		(instances
-			(project "USB-C-power-adapter"
+			(project "usb-c-power-adapter"
 				(path "/8da33aa8-79ed-467a-95ed-bf58aa0d1db6"
 					(page "2")
